File: PCB/GAS_SENSOR_I2C/untitled.brd (EAGLE design)
At the start: 44.6 x 21.6 mm, 40 parts, among them IC1 AZ1117CR2-5.0TRG1, IC2 LM393D, Q1 2N7002, Q2 2N7002, U2 LGT8F328P

Commit message: FEAT: update mq socket footprint
Parts:
- moved RST 2.16 mm to (30.6, 9.40)
- moved SWD 2.16 mm to (30.6, 10.9)
- moved 5V 1.52 mm to (30.6, 7.87)
- moved GND 1.52 mm to (30.6, 6.35)
- moved SWC 1.52 mm to (30.6, 12.4)
- moved U1 0.51 mm to (33.5, 9.53)
- moved C7 0.38 mm to (34.9, 9.40)
Routing:
- net IN1-: track 61.6 -> 76.7 mm, vias 1 -> 2
- net RESET: track 48.4 -> 38.5 mm, vias 4 -> 3
- net RX: track 34.0 -> 42.7 mm, vias 5 -> 6
- net TX: track 39.1 -> 45.5 mm, vias 8 -> 5
- net +5V: track 93.0 -> 97.5 mm
- net SWD: track 53.7 -> 51.1 mm, vias 5 -> 3
- net GND: track 11.7 -> 10.2 mm, vias 26 -> 23
- net SWC: track 36.3 -> 37.4 mm
